Commit message: formatting

File: urdf/elements.xacro (robot description, xacro)
@@ -6,20 +6,17 @@
         </geometry>
     </xacro:macro>
-    <xacro:macro
-        name="default_material">
+    <xacro:macro name="default_material">
         <material name="default_color">
             <color rgba="${48/255} ${213/255} ${200/255} 1" />
         </material>
     </xacro:macro>
-    <xacro:macro
-        name="param_material" params="r g b a">
+    <xacro:macro name="param_material" params="r g b a">
         <material name="param_color">
             <!-- TODO: Fix the color issue -->
-            <!-- *FIXED: It turned out the problem was Gazebo, not RViz -->
+            <!-- *FIXED: It turned out the problem was Gazebo, not RViz? -->
             <color rgba="${r/255} ${g/255} ${b/255} ${a}" />
         </material>
     </xacro:macro>
-    <xacro:macro
-        name="param_inertial" params="xyz rpy m ixx ixy ixz iyy iyz izz">
+    <xacro:macro name="param_inertial" params="xyz rpy m ixx ixy ixz iyy iyz izz">
         <inertial>
             <origin xyz="${xyz}" rpy="${rpy}" />
@@ -46,6 +43,5 @@
         </visual>
     </xacro:macro>
-    <xacro:macro
-        name="param_collision" params="xyz rpy stl">
+    <xacro:macro name="param_collision" params="xyz rpy stl">
         <collision>
             <origin xyz="${xyz}" rpy="${rpy}" />

File: urdf/joints.xacro (robot description, xacro)
@@ -9,6 +9,5 @@
         </joint>
     </xacro:macro>
-    <xacro:macro name="revolute_joint"
-        params="name parent child xyz rpy axis low up effort vel">
+    <xacro:macro name="revolute_joint" params="name parent child xyz rpy axis low up effort vel">
         <joint name="${name}" type="revolute">
             <origin xyz="${xyz}" rpy="${rpy}" />
@@ -19,6 +18,5 @@
         </joint>
     </xacro:macro>
-    <xacro:macro name="continuous_joint"
-        params="name parent child xyz rpy axis ">
+    <xacro:macro name="continuous_joint" params="name parent child xyz rpy axis ">
         <joint name="${name}" type="continuous">
             <origin xyz="${xyz}" rpy="${rpy}" />
@@ -56,6 +54,5 @@
     </xacro:macro>
     <!-- TODO: Make sure this doesn't cause problems -->
-    <xacro:macro name="support_wheel_axis_with_wheel"
-        params="prefix reflect">
+    <xacro:macro name="support_wheel_axis_with_wheel" params="prefix reflect">
         <xacro:fixed_joint name="joint_${prefix}_support_wheel_axis_with_wheel"
             parent="link_${prefix}_support_wheel_axis"
@@ -64,6 +61,5 @@
             rpy="0 0 0" />
     </xacro:macro>
-    <xacro:macro name="pedal_axis_with_pedal"
-        params="prefix reflect">
+    <xacro:macro name="pedal_axis_with_pedal" params="prefix reflect">
         <xacro:revolute_joint name="joint_${prefix}_pedal_axis_with_pedal"
             parent="link_${prefix}_pedal_axis"
@@ -80,6 +76,5 @@
     <!-- Moving this, make the whole bicycle moves (not the base_link though)-->
     <!-- joint_base_frame-->
-    <xacro:fixed_joint
-        name="joint_base_frame"
+    <xacro:fixed_joint name="joint_base_frame"
         parent="base_link"
         child="link_frame"
@@ -89,11 +84,9 @@
     <xacro:crank_arms_with_pedal_axis prefix="left" reflect="-1" />
     <!-- joint_crank_arms_right_pedal_axis -->
-    <xacro:crank_arms_with_pedal_axis
-        prefix="right" reflect="+1" />
+    <xacro:crank_arms_with_pedal_axis prefix="right" reflect="+1" />
     <!-- joint_left_support_leg_wheel_axis -->
     <xacro:support_leg_with_wheel_axis prefix="left" reflect="-1" />
     <!-- joint_right_support_leg_wheel_axis -->
-    <xacro:support_leg_with_wheel_axis
-        prefix="right" reflect="+1" />
+    <xacro:support_leg_with_wheel_axis prefix="right" reflect="+1" />
     <!-- joint_frame_crank_arms -->
     <xacro:revolute_joint name="joint_frame_crank_arms"
@@ -110,6 +103,5 @@
     <xacro:frame_with_support_leg prefix="left" reflect="-1" />
     <!-- joint_frame_right_support_leg -->
-    <xacro:frame_with_support_leg
-        prefix="right" reflect="+1" />
+    <xacro:frame_with_support_leg prefix="right" reflect="+1" />
     <!-- joint_frame_head_tube -->
     <xacro:revolute_joint name="joint_frame_head_tube"
@@ -135,6 +127,5 @@
         xyz="0 ${-0.425} ${-wheel_radius/2+0.03}"
         rpy="0 0 0"
-        axis="1 0 0"
-    />
+        axis="1 0 0" />
     <!-- joint_head_tube_handlebar -->
     <xacro:fixed_joint name="joint_head_tube_handlebar"
@@ -155,15 +146,12 @@
         xyz="0 ${-0.030} ${-0.46850}"
         rpy="${-20*PI/180} 0 0"
-        axis="1 0 0"
-    />
+        axis="1 0 0" />
     <!-- joint_left_support_wheel_axis_with_wheel -->
     <xacro:support_wheel_axis_with_wheel prefix="left" reflect="-1" />
     <!-- joint_right_support_wheel_axis_with_wheel -->
-    <xacro:support_wheel_axis_with_wheel
-        prefix="right" reflect="+1" />
+    <xacro:support_wheel_axis_with_wheel prefix="right" reflect="+1" />
     <!-- joint_left_pedal_axis_with_pedal -->
     <xacro:pedal_axis_with_pedal prefix="left" reflect="-1" />
     <!-- joint_right_pedal_axis_with_pedal -->
-    <xacro:pedal_axis_with_pedal
-        prefix="right" reflect="+1" />
+    <xacro:pedal_axis_with_pedal prefix="right" reflect="+1" />
 </robot>

File: urdf/lidar.xacro (robot description, xacro)
@@ -42,9 +42,15 @@
     </gazebo>
     <!-- frame_lidar_joint -->
-    <xacro:fixed_joint name="frame_lidar_joint" parent="link_frame" child="lidar_base_link"
-        xyz="0 0.41 0.25" rpy="0 0 0" />
+    <xacro:fixed_joint name="frame_lidar_joint"
+        parent="link_frame"
+        child="lidar_base_link"
+        xyz="0 0.41 0.25"
+        rpy="0 0 0" />
     <!-- base_lidar_joint -->
-    <xacro:fixed_joint name="base_lidar_joint" parent="lidar_base_link" child="link_lidar"
-        xyz="-.02 0 0.04" rpy="0 0 1.57" />
+    <xacro:fixed_joint name="base_lidar_joint"
+        parent="lidar_base_link"
+        child="link_lidar"
+        xyz="-.02 0 0.04"
+        rpy="0 0 1.57" />
     <!-- link_lidar plugin -->
     <gazebo reference="link_lidar">

File: urdf/links.xacro (robot description, xacro)
@@ -1,6 +1,5 @@
 <?xml version="1.0"?>
 <robot name="bicycle" xmlns:xacro="http://www.ros.org/wiki/xacro">
-    <xacro:macro
-        name="support_leg" params="prefix reflect">
+    <xacro:macro name="support_leg" params="prefix reflect">
         <link name="link_${prefix}_support_leg">
             <!-- Inertial -->
@@ -16,6 +15,5 @@
         </link>
     </xacro:macro>
-    <xacro:macro
-        name="support_wheel_axis" params="prefix reflect">
+    <xacro:macro name="support_wheel_axis" params="prefix reflect">
         <link name="link_${prefix}_support_wheel_axis">
             <!-- Inertial -->
@@ -32,6 +30,5 @@
         </link>
     </xacro:macro>
-    <xacro:macro
-        name="support_wheel" params="prefix reflect z">
+    <xacro:macro name="support_wheel" params="prefix reflect z">
         <link name="link_${prefix}_support_wheel">
             <!-- Inertial -->
@@ -63,6 +60,5 @@
     </link>
     <!-- link_back_wheel -->
-    <link
-        name="link_back_wheel">
+    <link name="link_back_wheel">
         <!-- Inertial -->
         <xacro:param_inertial xyz="0.04 0.09 0.5" rpy="0 0 0" m="1"
@@ -75,6 +71,5 @@
     </link>
     <!-- link_front_wheel -->
-    <link
-        name="link_front_wheel">
+    <link name="link_front_wheel">
         <!-- Inertial -->
         <xacro:param_inertial xyz="0.04 0.09 0" rpy="0 0 0" m="2"
@@ -87,6 +82,5 @@
     <!-- TODO: This was? considered a root link for some reason -->
     <!-- link_crank_arms -->
-    <link
-        name="link_crank_arms">
+    <link name="link_crank_arms">
         <!-- Inertial -->
         <xacro:param_inertial xyz="0 0 0" rpy="0 0 0" m="0.1"
@@ -98,6 +92,5 @@
     </link>
     <!-- link_left_pedal_axis -->
-    <link
-        name="link_left_pedal_axis">
+    <link name="link_left_pedal_axis">
         <!-- Inertial -->
         <xacro:param_inertial xyz="0 0 0" rpy="0 0 0" m="0.1"
@@ -111,6 +104,5 @@
     </link>
     <!-- link_right_pedal_axis -->
-    <link
-        name="link_right_pedal_axis">
+    <link name="link_right_pedal_axis">
         <!-- Inertial -->
         <xacro:param_inertial xyz="0 0 0" rpy="0 0 0" m="0.1"
@@ -124,6 +116,5 @@
     </link>
     <!-- link_left_pedal -->
-    <link
-        name="link_left_pedal">
+    <link name="link_left_pedal">
         <!-- Inertial -->
         <xacro:param_inertial xyz="0 0 0" rpy="0 0 0" m="0.1"
@@ -135,6 +126,5 @@
     </link>
     <!-- link_right_pedal -->
-    <link
-        name="link_right_pedal">
+    <link name="link_right_pedal">
         <!-- Inertial -->
         <xacro:param_inertial xyz="0 0 0" rpy="0 0 0" m="0.1"
@@ -146,6 +136,5 @@
     </link>
     <!-- link_fork -->
-    <link
-        name="link_fork">
+    <link name="link_fork">
         <!-- Inertial -->
         <xacro:param_inertial xyz="0 0 0" rpy="0 0 0" m="1"
@@ -159,6 +148,5 @@
     </link>
     <!-- link_head_tube -->
-    <link
-        name="link_head_tube">
+    <link name="link_head_tube">
         <!-- Inertial -->
         <xacro:param_inertial xyz="0 0 0" rpy="0 0 0" m="0.5"
@@ -173,6 +161,5 @@
     </link>
     <!-- link_handlebar -->
-    <link
-        name="link_handlebar">
+    <link name="link_handlebar">
         <!-- Inertial -->
         <xacro:param_inertial xyz="0 0 0" rpy="3.14159 1.55159 3.14159" m="0.5"
@@ -196,6 +183,5 @@
     <xacro:support_wheel prefix="right" reflect="+1" z="+1" />
     <!-- link_seat_post -->
-    <link
-        name="link_seat_post">
+    <link name="link_seat_post">
         <!-- Inertial -->
         <xacro:param_inertial xyz="0 0 0" rpy="1.59 0 0" m="0.5"
