Commit message: add gazebo material

File: urdf/gazebo_config.xacro (robot description, xacro)
@@ -14,4 +14,49 @@
         <material>Gazebo/Turquoise</material>
     </gazebo>
+    <gazebo reference="link_fork">
+        <material>Gazebo/Turquoise</material>
+    </gazebo>
+    <gazebo reference="link_head_tube">
+        <material>Gazebo/Black</material>
+    </gazebo>
+    <gazebo reference="link_handlebar">
+        <material>Gazebo/Black</material>
+    </gazebo>
+    <gazebo reference="link_crank_arms">
+        <material>Gazebo/Black</material>
+    </gazebo>
+    <gazebo reference="link_left_support_wheel_axis">
+        <material>Gazebo/White</material>
+    </gazebo>
+    <gazebo reference="link_right_support_wheel_axis">
+        <material>Gazebo/White</material>
+    </gazebo>
+    <gazebo reference="link_left_support_wheel">
+        <material>Gazebo/White</material>
+    </gazebo>
+    <gazebo reference="link_right_support_wheel">
+        <material>Gazebo/White</material>
+    </gazebo>
+    <gazebo reference="link_left_support_leg">
+        <material>Gazebo/White</material>
+    </gazebo>
+    <gazebo reference="link_right_support_leg">
+        <material>Gazebo/White</material>
+    </gazebo>
+    <gazebo reference="link_seat_post">
+        <material>Gazebo/Black</material>
+    </gazebo>
+    <gazebo reference="link_left_pedal_axis">
+        <material>Gazebo/Black</material>
+    </gazebo>
+    <gazebo reference="link_right_pedal_axis">
+        <material>Gazebo/Black</material>
+    </gazebo>
+    <gazebo reference="link_left_pedal">
+        <material>Gazebo/Black</material>
+    </gazebo>
+    <gazebo reference="link_right_pedal">
+        <material>Gazebo/Black</material>
+    </gazebo>
     <gazebo reference="link_back_wheel">
         <material>Gazebo/Black</material>

Commit message: move lidar link color to lidar.xacro

File: urdf/gazebo_config.xacro (robot description, xacro)
@@ -65,9 +65,3 @@
         <material>Gazebo/Black</material>
     </gazebo>
-    <gazebo reference="link_lidar">
-        <material>Gazebo/Black</material>
-    </gazebo>
-    <gazebo reference="lidar_base_link">
-        <material>Gazebo/Red</material>
-    </gazebo>
 </robot>

Commit message: fix material issue

File: urdf/gazebo_config.xacro (robot description, xacro)
@@ -2,10 +2,12 @@
 <robot name="bicycle" xmlns:xacro="http://www.ros.org/wiki/xacro">
     <gazebo reference="link_left_support_wheel">
-        <material>Gazebo/Black</material>
         <mu1 value="1e-3" />
         <mu2 value="1e-3" />
     </gazebo>
     <gazebo reference="link_right_support_wheel">
-        <material>Gazebo/Black</material>
+        <mu1 value="1e-3" />
+        <mu2 value="1e-3" />
+    </gazebo>
+    <gazebo reference="link_front_wheel">
         <mu1 value="1e-3" />
         <mu2 value="1e-3" />
