Commit message: edited mass values

File: urdf/property.xacro (robot description, xacro)
@@ -5,14 +5,14 @@
     <xacro:property name="wheel_thickness" value="0.05" />
     <xacro:property name="wheel_separation" value="0.98" />
-    <xacro:property name="wheel_mass" value="0.5" />
-    <xacro:property name="support_leg_mass" value="0.1" />
+    <xacro:property name="wheel_mass" value="1.0" />
+    <xacro:property name="support_leg_mass" value="0.3" />
     <xacro:property name="support_axis_mass" value="0.1" />
-    <xacro:property name="support_wheel_mass" value="0.1" />
+    <xacro:property name="support_wheel_mass" value="0.5" />
     <xacro:property name="frame_offset_z" value="${2*wheel_radius+const_1}" />
-    <xacro:property name="frame_mass" value="0.1" />
-    <xacro:property name="screw_mass" value="0.1" />
-    <xacro:property name="seat_stay_mass" value="0.1" />
-    <xacro:property name="fork_mass" value="0.1" />
-    <xacro:property name="head_tube_mass" value="0.1" />
+    <xacro:property name="frame_mass" value="1.5" />
+    <xacro:property name="screw_mass" value="0.2" />
+    <xacro:property name="seat_stay_mass" value="0.5" />
+    <xacro:property name="fork_mass" value="0.5" />
+    <xacro:property name="head_tube_mass" value="0.2" />
     <xacro:property name="const_1" value="0.10" />
     <xacro:property name="cylindar_radius" value="0.01" />

Commit message: changed wheel_thickness

File: urdf/property.xacro (robot description, xacro)
@@ -4,5 +4,6 @@
     <!-- TODO: thickns wheels -->
     <xacro:property name="wheel_radius" value="0.25" />
-    <xacro:property name="wheel_thickness" value="0.05" />
+    <!-- <xacro:property name="wheel_thickness" value="0.05" /> -->
+    <xacro:property name="wheel_thickness" value="0.1" />
     <xacro:property name="wheel_separation" value="0.98" />
     <xacro:property name="wheel_mass" value="1.0" />
