Commit message: added bicycle control

File: urdf/ros2_control.xacro (robot description, xacro)
@@ -17,5 +17,6 @@
             <state_interface name="position" />
         </joint>
-        <joint name="joint_frame_head_tube">
+        <!-- <joint name="joint_frame_head_tube"> -->
+        <joint name="joint_fork_front_wheel">
             <command_interface name="position">
                 <param name="initial_value">0.0</param>

Commit message: added frame_head_joint

File: urdf/ros2_control.xacro (robot description, xacro)
@@ -5,4 +5,16 @@
             <plugin>gazebo_ros2_control/GazeboSystem</plugin>
         </hardware>
+        <joint name="frame_head_joint">
+            <command_interface name="position">
+                <param name="min">-1.570796327</param>
+                <param name="max">+1.570796327</param>
+            </command_interface>
+            <command_interface name="velocity">
+                <param name="min">-0.1</param>
+                <param name="max">+0.1</param>
+            </command_interface>
+            <state_interface name="position" />
+            <state_interface name="velocity" />
+        </joint>
         <joint name="screw_front_wheel_joint">
             <command_interface name="position">
@@ -11,6 +23,6 @@
             </command_interface>
             <command_interface name="velocity">
-                <param name="min">-10</param>
-                <param name="max">10</param>
+                <param name="min">-1</param>
+                <param name="max">+1</param>
             </command_interface>
             <state_interface name="position" />
@@ -18,11 +30,11 @@
         </joint>
         <joint name="screw_back_wheel_joint">
-            <command_interface name="position">
+            <!-- <command_interface name="position">
                 <param name="min">-3.1415</param>
                 <param name="max">3.1415</param>
-            </command_interface>
+            </command_interface> -->
             <command_interface name="velocity">
-                <param name="min">-10</param>
-                <param name="max">10</param>
+                <param name="min">-1</param>
+                <param name="max">+1</param>
             </command_interface>
             <state_interface name="position" />

Commit message: added sim_mode

File: urdf/ros2_control.xacro (robot description, xacro)
@@ -1,34 +1,42 @@
 <?xml version="1.0"?>
 <robot name="bicycle" xmlns:xacro="http://www.ros.org/wiki/xacro">
-    <ros2_control name="GazeboSystem" type="system">
-        <hardware>
-            <plugin>gazebo_ros2_control/GazeboSystem</plugin>
-        </hardware>
-        <joint name="frame_head_joint">
-            <command_interface name="position">
-                <param name="min">-1.570796327</param>
-                <param name="max">+1.570796327</param>
-            </command_interface>
-            <state_interface name="position" />
-        </joint>
-        <joint name="screw_front_wheel_joint">
-            <command_interface name="position">
-                <param name="min">-1.570796327</param>
-                <param name="max">+1.570796327</param>
-            </command_interface>
-            <state_interface name="position" />
-        </joint>
-        <joint name="screw_back_wheel_joint">
-            <command_interface name="velocity">
-                <param name="min">-1</param>
-                <param name="max">+1</param>
-            </command_interface>
-            <state_interface name="position" />
-            <state_interface name="velocity" />
-        </joint>
-    </ros2_control>
+    <!-- TODO: Add hardware interface plugin here, and configure it -->
+    <xacro:unless value="$(arg sim_mode)">
+    </xacro:unless>
+    <xacro:if value="$(arg sim_mode)">
+        <ros2_control name="GazeboSystem" type="system">
+            <hardware>
+                <plugin>gazebo_ros2_control/GazeboSystem</plugin>
+            </hardware>
+            <joint name="frame_head_joint">
+                <command_interface name="position">
+                    <param name="min">-1.570796327</param>
+                    <param name="max">+1.570796327</param>
+                </command_interface>
+                <state_interface name="position" />
+            </joint>
+            <joint name="screw_front_wheel_joint">
+                <command_interface name="position">
+                    <param name="min">-1.570796327</param>
+                    <param name="max">+1.570796327</param>
+                </command_interface>
+                <state_interface name="position" />
+            </joint>
+            <joint name="screw_back_wheel_joint">
+                <command_interface name="velocity">
+                    <param name="min">-1</param>
+                    <param name="max">+1</param>
+                </command_interface>
+                <state_interface name="position" />
+                <state_interface name="velocity" />
+            </joint>
+        </ros2_control>
+    </xacro:if>
     <gazebo>
         <plugin name="gazebo_ros2_control" filename="libgazebo_ros2_control.so">
             <parameters>$(find bicycle_sim)/config/bicycle_controllers.yaml</parameters>
+            <!-- TODO: You may have to git clone to src -->
+            <!-- git clone -b humble https://github.com/ros-controls/gazebo_ros2_control -->
+            <!-- <parameters>$(find bicycle_sim)/config/gazebo_sim_mode.yaml</parameters> -->
         </plugin>
     </gazebo>
