Commit message: urdf structure change

File: urdf/bicycle.urdf.xacro (robot description, xacro)
@@ -7,14 +7,6 @@
   <!-- PROPERTIES -->
   <xacro:include filename="properties.xacro" />
-  <!-- JOINTS TYPE-->
-  <xacro:include filename="joints_type.xacro" />
   <!-- ELEMENTS -->
   <xacro:include filename="elements.xacro" />
-  <!-- BICYCLE JOINTS -->
-  <xacro:include filename="bicycle_joints.xacro" />
-  <!-- BICYCLE LINKS -->
-  <xacro:include filename="bicycle_links.xacro" />
-  <!-- GAZEBO -->
-  <!-- <xacro:include filename="gazebo.xacro" /> -->
   <!-- ========================LINKS======================== -->
   <xacro:include filename="links.xacro" />
@@ -22,11 +14,8 @@
   <xacro:include filename="joints.xacro" />
   <!-- ========================GAZEBO======================== -->
-  <!-- Here, we link Gazebo to the ROS library. -->
-  <!-- <xacro:include filename="gazebo_ros.xacro" /> -->
-  <!-- GAZEBO COLORS -->
   <xacro:include filename="gazebo_config.xacro" />
   <!-- ====================LiDAR SANNER=================== -->
   <xacro:include filename="lidar.xacro" />
   <!-- ====================CAMERA=================== -->
-  <xacro:include filename="camera.xacro" />
+  <!-- <xacro:include filename="camera.xacro" /> -->
 </robot>

File: urdf/joints.xacro (robot description, xacro)
@@ -1,4 +1,80 @@
 <?xml version="1.0"?>
 <robot name="bicycle" xmlns:xacro="http://www.ros.org/wiki/xacro">
+    <xacro:macro name="fixed_joint" params="name parent child xyz rpy">
+        <joint name="${name}" type="fixed">
+            <origin xyz="${xyz}" rpy="${rpy}" />
+            <parent link="${parent}" />
+            <child link="${child}" />
+        </joint>
+    </xacro:macro>
+    <xacro:macro name="revolute_joint"
+        params="name parent child xyz rpy axis low up effort vel">
+        <joint name="${name}" type="revolute">
+            <origin xyz="${xyz}" rpy="${rpy}" />
+            <parent link="${parent}" />
+            <child link="${child}" />
+            <axis xyz="${axis}" />
+            <limit lower="${low}" upper="${up}" effort="${effort}" velocity="${vel}" />
+        </joint>
+    </xacro:macro>
+    <xacro:macro name="continuous_joint"
+        params="name parent child xyz rpy axis ">
+        <joint name="${name}" type="continuous">
+            <origin xyz="${xyz}" rpy="${rpy}" />
+            <parent link="${parent}" />
+            <child link="${child}" />
+            <axis xyz="${axis}" />
+        </joint>
+    </xacro:macro>
+    <!-- ===================================================================== -->
+    <xacro:macro name="crank_arms_with_pedal_axis" params="prefix reflect">
+        <xacro:fixed_joint name="joint_crank_arms_${prefix}_pedal_axis"
+            parent="link_crank_arms"
+            child="link_${prefix}_pedal_axis"
+            xyz="${reflect*0.070} 0 ${reflect*0.1750}"
+            rpy="0 0 0" />
+    </xacro:macro>
+    <xacro:macro name="support_leg_with_wheel_axis" params="prefix reflect">
+        <xacro:revolute_joint name="joint_${prefix}_support_leg_wheel_axis"
+            parent="link_${prefix}_support_leg"
+            child="link_${prefix}_support_wheel_axis"
+            xyz="${reflect*0.105} 0 ${-wheel_radius+support_wheel_radius}"
+            rpy="0 0 0"
+            axis="1 0 0"
+            low="-${PI}"
+            up="${PI}"
+            effort="10"
+            vel="10" />
+    </xacro:macro>
+    <xacro:macro name="frame_with_support_leg" params="prefix reflect">
+        <xacro:fixed_joint name="joint_frame_${prefix}_support_leg"
+            parent="link_frame"
+            child="link_${prefix}_support_leg"
+            xyz="0 ${-0.425} ${-0.1}"
+            rpy="0 0 0" />
+    </xacro:macro>
+    <!-- TODO: Make sure this doesn't cause problems -->
+    <xacro:macro name="support_wheel_axis_with_wheel"
+        params="prefix reflect">
+        <xacro:fixed_joint name="joint_${prefix}_support_wheel_axis_with_wheel"
+            parent="link_${prefix}_support_wheel_axis"
+            child="link_${prefix}_support_wheel"
+            xyz="0 0 0"
+            rpy="0 0 0" />
+    </xacro:macro>
+    <xacro:macro name="pedal_axis_with_pedal"
+        params="prefix reflect">
+        <xacro:revolute_joint name="joint_${prefix}_pedal_axis_with_pedal"
+            parent="link_${prefix}_pedal_axis"
+            child="link_${prefix}_pedal"
+            xyz="${reflect*0.100} 0 0"
+            rpy="0 0 0"
+            axis="1 0 0"
+            low="-${PI}"
+            up="${PI}"
+            effort="10"
+            vel="10" />
+    </xacro:macro>
+    <!-- ===================================================================== -->
     <!-- Moving this, make the whole bicycle moves (not the base_link though)-->
     <!-- joint_base_frame-->

File: urdf/links.xacro (robot description, xacro)
@@ -1,12 +1,53 @@
 <?xml version="1.0"?>
 <robot name="bicycle" xmlns:xacro="http://www.ros.org/wiki/xacro">
-    <!-- world-->
-    <!-- <link name="world" /> -->
+    <xacro:macro
+        name="support_leg" params="prefix reflect">
+        <link name="link_${prefix}_support_leg">
+            <!-- Inertial -->
+            <xacro:param_inertial xyz="0 0 0" rpy="0 0 0" m="0.5"
+                ixx="0.166667" ixy="0" ixz="0" iyy="0.166667" iyz="0" izz="0.166667" />
+            <!-- Visual -->
+            <xacro:param_visual xyz="${reflect*0.215} ${-reflect*0.018} ${-0.12}"
+                rpy="${-PI/2} 0 ${reflect*PI/2}" stl="link_${prefix}_support_leg"
+                r="0" g="0" b="0" a="1" />
+            <!-- Collision -->
+            <xacro:param_collision xyz="${reflect*0.215} ${-reflect*0.018} ${-0.12}"
+                rpy="1.57 ${PI} ${-reflect*PI/2}" stl="link_${prefix}_support_leg" />
+        </link>
+    </xacro:macro>
+    <xacro:macro
+        name="support_wheel_axis" params="prefix reflect">
+        <link name="link_${prefix}_support_wheel_axis">
+            <!-- Inertial -->
+            <xacro:param_inertial xyz="0 0 0" rpy="3.14159 1.55159 3.14159" m="0.5"
+                ixx="0.166667" ixy="0" ixz="0" iyy="0.166667" iyz="0" izz="0.166667" />
+            <!-- Visual -->
+            <!-- TODO: Make sure it fits with support wheels-->
+            <xacro:param_visual xyz="${reflect*0.035} 0 0" rpy="0 ${-reflect*PI/2} 0"
+                stl="link_${prefix}_support_wheel_axis"
+                r="0" g="0" b="0" a="1" />
+            <!-- Collision -->
+            <xacro:param_collision xyz="${reflect*0.035} 0 0" rpy="0 ${-reflect*PI/2} 0"
+                stl="link_${prefix}_support_wheel_axis" />
+        </link>
+    </xacro:macro>
+    <xacro:macro
+        name="support_wheel" params="prefix reflect z">
+        <link name="link_${prefix}_support_wheel">
+            <!-- Inertial -->
+            <xacro:param_inertial xyz="0 0 0" rpy="0 0 0" m="1"
+                ixx="0.166667" ixy="0" ixz="0" iyy="0.166667" iyz="0" izz="0.166667" />
+            <!-- Visual -->
+            <xacro:param_visual xyz="${reflect*0.035} 0 0" rpy="0 0 ${z*PI}"
+                stl="link_${prefix}_support_wheel"
+                r="255" g="255" b="255" a="1" />
+            <!-- Collision -->
+            <xacro:param_collision xyz="${reflect*0.035} 0 0" rpy="0 0 ${z*PI}"
+                stl="link_${prefix}_support_wheel" />
+        </link>
+    </xacro:macro>
+    <!-- ===================================================================== -->
     <!-- base_link -->
     <link name="base_link" />
-    <!-- <joint name="world_base" type="fixed">
-    <parent link="world" />
-    <child link="base_link" />
-  </joint> -->
     <!--link_frame-->
     <link name="link_frame">
@@ -44,5 +85,5 @@
         <xacro:param_collision xyz="0 0 0" rpy="0 0 0" stl="link_front_wheel" />
     </link>
-    <!-- TODO: This is considered a root link for some reason -->
+    <!-- TODO: This was? considered a root link for some reason -->
     <!-- link_crank_arms -->
     <link
@@ -143,16 +184,13 @@
     </link>
     <!-- link_left_support_leg -->
-    <xacro:support_leg
-        prefix="left" reflect="-1" />
+    <xacro:support_leg prefix="left" reflect="-1" />
     <!-- link_right_support_leg -->
     <xacro:support_leg prefix="right" reflect="+1" />
     <!-- link_left_support_wheel_axis -->
-    <xacro:support_wheel_axis
-        prefix="left" reflect="-1" />
+    <xacro:support_wheel_axis prefix="left" reflect="-1" />
     <!-- link_right_support_wheel_axis -->
     <xacro:support_wheel_axis prefix="right" reflect="+1" />
     <!-- link_left_support_wheel -->
-    <xacro:support_wheel
-        prefix="left" reflect="-1" z="0" />
+    <xacro:support_wheel prefix="left" reflect="-1" z="0" />
     <!-- link_right_support_wheel -->
     <xacro:support_wheel prefix="right" reflect="+1" z="+1" />
