Commit message: added ros2_control

File: urdf/bicycle.urdf.xacro (robot description, xacro)
@@ -1,23 +1,504 @@
 <?xml version="1.0"?>
 <robot name="bicycle" xmlns:xacro="http://www.ros.org/wiki/xacro">
-  <!-- TODO: Calculate the inertia matrix -->
-  <!-- TODO: Make sure joints type are valid for simulation (Gazebo) -->
-  <!-- TODO: Simpler collision -->
-  <!-- ========================MACROS======================== -->
-  <!-- PROPERTIES -->
-  <xacro:include filename="properties.xacro" />
-  <!-- ELEMENTS -->
-  <xacro:include filename="elements.xacro" />
-  <!-- ========================LINKS======================== -->
-  <xacro:include filename="links.xacro" />
-  <!-- ========================JOINTS======================== -->
-  <xacro:include filename="joints.xacro" />
-  <!-- ========================ros2_control======================== -->
-  <!-- <xacro:include filename="ros2_control.xacro" /> -->
-  <!-- ========================GAZEBO======================== -->
-  <xacro:include filename="gazebo_config.xacro" />
-  <!-- ====================LiDAR SANNER=================== -->
-  <xacro:include filename="lidar.xacro" />
-  <!-- ====================CAMERA=================== -->
-  <!-- <xacro:include filename="camera.xacro" /> -->
+    <xacro:include filename="material.xacro" />
+    <xacro:include filename="property.xacro" />
+    <xacro:include filename="inertial.xacro" />
+    <xacro:include filename="ros2_control.xacro" />
+    <!-- BASE LINK -->
+    <link name="base_link" />
+    <!-- BASE FOOTPRINT LINK -->
+    <joint name="base_footprint_joint" type="fixed">
+        <parent link="base_link" />
+        <child link="base_footprint" />
+        <origin xyz="0 0 0" rpy="0 0 0" />
+    </joint>
+    <link name="base_footprint" />
+    <!-- FRAME LINK -->
+    <joint name="base_frame_joint" type="fixed">
+        <parent link="base_link" />
+        <child link="frame" />
+        <origin xyz="0 0 ${frame_offset_z}" rpy="0 0 0" />
+    </joint>
+    <link name="frame">
+        <visual>
+            <origin xyz="0 0 0" rpy="${pi/2} 0 0" />
+            <geometry>
+                <cylinder length="${wheel_separation}" radius="${cylindar_radius}" />
+            </geometry>
+            <material name="cyan" />
+        </visual>
+        <collision>
+            <origin xyz="0 0 0" rpy="${pi/2} 0 0" />
+            <geometry>
+                <cylinder length="${wheel_separation}" radius="${cylindar_radius}" />
+            </geometry>
+        </collision>
+        <xacro:inertial_cylinder mass="${frame_mass}" length="${wheel_separation}"
+            radius="${cylindar_radius}">
+            <origin xyz="0 0 0" rpy="${pi/2} 0 0" />
+        </xacro:inertial_cylinder>
+    </link>
+    <gazebo reference="frame">
+        <material>Gazebo/Turquoise</material>
+    </gazebo>
+    <!-- HEAD TUBE LINK -->
+    <joint name="frame_head_joint" type="revolute">
+        <axis xyz="1 0 0" />
+        <limit effort="10" lower="-1.570796327" upper="+1.570796327" velocity="10" />
+        <parent link="frame" />
+        <child link="head_tube" />
+        <origin xyz="0 ${wheel_separation/2} 0" rpy="0 ${pi/2} 0" />
+    </joint>
+    <link name="head_tube">
+        <visual>
+            <origin xyz="0 0 0" rpy="0 0 0" />
+            <geometry>
+                <cylinder length="${2*wheel_thickness}" radius="${cylindar_radius}" />
+            </geometry>
+            <material name="white" />
+        </visual>
+        <collision>
+            <origin xyz="0 0 0" rpy="0 0 0" />
+            <geometry>
+                <cylinder length="${2*wheel_thickness}" radius="${cylindar_radius}" />
+            </geometry>
+        </collision>
+        <xacro:inertial_cylinder mass="${head_tube_mass}" length="${2*wheel_thickness}"
+            radius="${cylindar_radius}">
+            <origin xyz="0 0 0" rpy="0 0 0" />
+        </xacro:inertial_cylinder>
+    </link>
+    <gazebo reference="head_tube">
+        <material>Gazebo/White</material>
+    </gazebo>
+    <!-- BACK HEAD TUBE LINK -->
+    <joint name="frame_back_head_joint" type="fixed">
+        <parent link="frame" />
+        <child link="back_head_tube" />
+        <origin xyz="0 ${-wheel_separation/2} 0" rpy="0 ${pi/2} 0" />
+    </joint>
+    <link name="back_head_tube">
+        <visual>
+            <origin xyz="0 0 0" rpy="0 0 0" />
+            <geometry>
+                <cylinder length="${2*wheel_thickness}" radius="${cylindar_radius}" />
+            </geometry>
+            <material name="white" />
+        </visual>
+        <collision>
+            <origin xyz="0 0 0" rpy="0 0 0" />
+            <geometry>
+                <cylinder length="${2*wheel_thickness}" radius="${cylindar_radius}" />
+            </geometry>
+        </collision>
+        <xacro:inertial_cylinder mass="${head_tube_mass}" length="${2*wheel_thickness}"
+            radius="${cylindar_radius}">
+            <origin xyz="0 0 0" rpy="0 0 0" />
+        </xacro:inertial_cylinder>
+    </link>
+    <gazebo reference="back_head_tube">
+        <material>Gazebo/White</material>
+    </gazebo>
+    <!-- FORK RIGHT LINK -->
+    <joint name="head_fork_right_joint" type="fixed">
+        <parent link="head_tube" />
+        <child link="fork_right" />
+        <origin xyz="0 0 ${wheel_thickness}" rpy="0 ${-pi/2} 0" />
+    </joint>
+    <link name="fork_right">
+        <visual>
+            <origin xyz="0 0 ${-(wheel_radius+const_1)/2}" rpy="0 0 0" />
+            <geometry>
+                <cylinder length="${wheel_radius+const_1}" radius="${cylindar_radius}" />
+            </geometry>
+            <material name="cyan" />
+        </visual>
+        <collision>
+            <origin xyz="0 0 ${-(wheel_radius+const_1)/2}" rpy="0 0 0" />
+            <geometry>
+                <cylinder length="${wheel_radius+const_1}" radius="${cylindar_radius}" />
+            </geometry>
+        </collision>
+        <xacro:inertial_cylinder mass="${fork_mass}" length="${wheel_radius+const_1}"
+            radius="${cylindar_radius}">
+            <origin xyz="0 0 ${-(wheel_radius+const_1)/2}" rpy="0 0 0" />
+        </xacro:inertial_cylinder>
+    </link>
+    <gazebo reference="fork_right">
+        <material>Gazebo/Turquoise</material>
+    </gazebo>
+    <!-- FORK LEFT LINK -->
+    <joint name="head_fork_left_joint" type="fixed">
+        <parent link="head_tube" />
+        <child link="fork_left" />
+        <origin xyz="0 0 ${-wheel_thickness}" rpy="0 ${-pi/2} 0" />
+    </joint>
+    <link name="fork_left">
+        <visual>
+            <origin xyz="0 0 ${-(wheel_radius+const_1)/2}" rpy="0 0 0" />
+            <geometry>
+                <cylinder length="${wheel_radius+const_1}" radius="${cylindar_radius}" />
+            </geometry>
+            <material name="cyan" />
+        </visual>
+        <collision>
+            <origin xyz="0 0 ${-(wheel_radius+const_1)/2}" rpy="0 0 0" />
+            <geometry>
+                <cylinder length="${wheel_radius+const_1}" radius="${cylindar_radius}" />
+            </geometry>
+        </collision>
+        <xacro:inertial_cylinder mass="${fork_mass}" length="${wheel_radius+const_1}"
+            radius="${cylindar_radius}">
+            <origin xyz="0 0 ${-(wheel_radius+const_1)/2}" rpy="0 0 0" />
+        </xacro:inertial_cylinder>
+    </link>
+    <gazebo reference="fork_left">
+        <material>Gazebo/Turquoise</material>
+    </gazebo>
+    <!-- FRONT SCREW LINK -->
+    <joint name="head_back_screw_joint" type="fixed">
+        <parent link="head_tube" />
+        <child link="front_screw" />
+        <origin xyz="${wheel_radius+const_1} 0 0" rpy="0 0 0" />
+    </joint>
+    <link name="front_screw">
+        <visual>
+            <origin xyz="0 0 0" rpy="0 0 0" />
+            <geometry>
+                <cylinder length="${2*wheel_thickness}" radius="${cylindar_radius}" />
+            </geometry>
+            <material name="white" />
+        </visual>
+        <collision>
+            <origin xyz="0 0 0" rpy="0 0 0" />
+            <geometry>
+                <cylinder length="${2*wheel_thickness}" radius="${cylindar_radius}" />
+            </geometry>
+        </collision>
+        <xacro:inertial_cylinder mass="${screw_mass}" length="${2*wheel_thickness}"
+            radius="${cylindar_radius}">
+            <origin xyz="0 0 0" rpy="0 0 0" />
+        </xacro:inertial_cylinder>
+    </link>
+    <gazebo reference="front_screw">
+        <material>Gazebo/White</material>
+    </gazebo>
+    <!-- SEAT STAY LEFT LINK -->
+    <joint name="back_head_seat_left_joint" type="fixed">
+        <parent link="back_head_tube" />
+        <child link="seat_stay_left" />
+        <origin xyz="0 0 ${-wheel_thickness}" rpy="0 ${-pi/2} 0" />
+    </joint>
+    <link name="seat_stay_left">
+        <visual>
+            <origin xyz="0 0 ${-(wheel_radius+const_1)/2}" rpy="0 0 0" />
+            <geometry>
+                <cylinder length="${wheel_radius+const_1}" radius="${cylindar_radius}" />
+            </geometry>
+            <material name="cyan" />
+        </visual>
+        <collision>
+            <origin xyz="0 0 ${-(wheel_radius+const_1)/2}" rpy="0 0 0" />
+            <geometry>
+                <cylinder length="${wheel_radius+const_1}" radius="${cylindar_radius}" />
+            </geometry>
+        </collision>
+        <xacro:inertial_cylinder mass="${seat_stay_mass}" length="${wheel_radius+const_1}"
+            radius="${cylindar_radius}">
+            <origin xyz="0 0 ${-(wheel_radius+const_1)/2}" rpy="0 0 0" />
+        </xacro:inertial_cylinder>
+    </link>
+    <gazebo reference="seat_stay_left">
+        <material>Gazebo/Turquoise</material>
+    </gazebo>
+    <!-- SEAT STAY RIGHT LINK -->
+    <joint name="back_head_seat_right_joint" type="fixed">
+        <parent link="back_head_tube" />
+        <child link="seat_stay_right" />
+        <origin xyz="0 0 ${+wheel_thickness}" rpy="0 ${-pi/2} 0" />
+    </joint>
+    <link name="seat_stay_right">
+        <visual>
+            <origin xyz="0 0 ${-(wheel_radius+const_1)/2}" rpy="0 0 0" />
+            <geometry>
+                <cylinder length="${wheel_radius+const_1}" radius="${cylindar_radius}" />
+            </geometry>
+            <material name="cyan" />
+        </visual>
+        <collision>
+            <origin xyz="0 0 ${-(wheel_radius+const_1)/2}" rpy="0 0 0" />
+            <geometry>
+                <cylinder length="${wheel_radius+const_1}" radius="${cylindar_radius}" />
+            </geometry>
+        </collision>
+        <xacro:inertial_cylinder mass="${seat_stay_mass}" length="${wheel_radius+const_1}"
+            radius="${cylindar_radius}">
+            <origin xyz="0 0 ${-(wheel_radius+const_1)/2}" rpy="0 0 0" />
+        </xacro:inertial_cylinder>
+    </link>
+    <gazebo reference="seat_stay_right">
+        <material>Gazebo/Turquoise</material>
+    </gazebo>
+    <!-- BACK SCREW LINK -->
+    <joint name="back_head_back_screw_joint" type="fixed">
+        <parent link="back_head_tube" />
+        <child link="back_screw" />
+        <origin xyz="${wheel_radius+const_1} 0 0" rpy="0 0 0" />
+    </joint>
+    <link name="back_screw">
+        <visual>
+            <origin xyz="0 0 0" rpy="0 0 0" />
+            <geometry>
+                <cylinder length="${2*wheel_thickness}" radius="${cylindar_radius}" />
+            </geometry>
+            <material name="white" />
+        </visual>
+        <collision>
+            <origin xyz="0 0 0" rpy="0 0 0" />
+            <geometry>
+                <cylinder length="${2*wheel_thickness}" radius="${cylindar_radius}" />
+            </geometry>
+        </collision>
+        <xacro:inertial_cylinder mass="${screw_mass}" length="${2*wheel_thickness}"
+            radius="${cylindar_radius}">
+            <origin xyz="0 0 0" rpy="0 0 0" />
+        </xacro:inertial_cylinder>
+    </link>
+    <gazebo reference="back_screw">
+        <material>Gazebo/White</material>
+    </gazebo>
+    <!-- FRONT WHEEL -->
+    <joint name="screw_front_wheel_joint" type="continuous">
+        <axis xyz="0 0 1" />
+        <!-- <parent link="base_link" /> -->
+        <parent link="front_screw" />
+        <child link="front_wheel" />
+        <origin xyz="0 0 0" rpy="0 ${-pi} 0" />
+    </joint>
+    <link name="front_wheel">
+        <visual>
+            <origin xyz="0 0 0" rpy="0 0 0" />
+            <geometry>
+                <cylinder length="${wheel_thickness}" radius="${wheel_radius}" />
+            </geometry>
+            <material name="black" />
+        </visual>
+        <collision>
+            <origin xyz="0 0 0" rpy="0 0 0" />
+            <geometry>
+                <sphere radius="${wheel_radius}" />
+            </geometry>
+        </collision>
+        <xacro:inertial_cylinder mass="${wheel_mass}" length="${wheel_thickness}"
+            radius="${wheel_radius}">
+            <origin xyz="0 0 0" rpy="0 0 0" />
+        </xacro:inertial_cylinder>
+    </link>
+    <gazebo reference="front_wheel">
+        <material>Gazebo/Black</material>
+    </gazebo>
+    <!-- BACK WHEEL -->
+    <joint name="screw_back_wheel_joint" type="continuous">
+        <axis xyz="0 0 1" />
+        <!-- <parent link="base_link" /> -->
+        <parent link="back_screw" />
+        <child link="back_wheel" />
+        <origin xyz="0 0 0" rpy="0 ${-pi} 0" />
+    </joint>
+    <link name="back_wheel">
+        <visual>
+            <origin xyz="0 0 0" rpy="0 0 0" />
+            <geometry>
+                <cylinder length="${wheel_thickness}" radius="${wheel_radius}" />
+            </geometry>
+            <material name="black" />
+        </visual>
+        <collision>
+            <origin xyz="0 0 0" rpy="0 0 0" />
+            <geometry>
+                <sphere radius="${wheel_radius}" />
+            </geometry>
+        </collision>
+        <xacro:inertial_cylinder mass="${wheel_mass}" length="${wheel_thickness}"
+            radius="${wheel_radius}">
+            <origin xyz="0 0 0" rpy="0 0 0" />
+        </xacro:inertial_cylinder>
+    </link>
+    <gazebo reference="back_wheel">
+        <material>Gazebo/Black</material>
+    </gazebo>
+    <!-- RIGHT SUPPORT LEG LINK -->
+    <joint name="screw_right_support_joint" type="fixed">
+        <parent link="back_screw" />
+        <child link="right_support_leg" />
+        <origin xyz="0 0 ${wheel_thickness}" rpy="0 ${-pi/2} 0" />
+    </joint>
+    <link name="right_support_leg">
+        <visual>
+            <origin xyz="0 0 ${-3/8*wheel_radius}" rpy="0 0 0" />
+            <geometry>
+                <cylinder length="${3/4*wheel_radius}" radius="${cylindar_radius}" />
+            </geometry>
+            <material name="white" />
+        </visual>
+        <collision>
+            <origin xyz="0 0 ${-3/8*wheel_radius}" rpy="0 0 0" />
+            <geometry>
+                <cylinder length="${3/4*wheel_radius}" radius="${cylindar_radius}" />
+            </geometry>
+        </collision>
+        <xacro:inertial_cylinder mass="${support_leg_mass}" length="${3/4*wheel_radius}"
+            radius="${cylindar_radius}">
+            <origin xyz="0 0 ${-3/8*wheel_radius}" rpy="0 0 0" />
+        </xacro:inertial_cylinder>
+    </link>
+    <gazebo reference="right_support_leg">
+        <material>Gazebo/White</material>
+    </gazebo>
+    <!-- RIGHT SUPPORT AXIS LINK -->
+    <joint name="right_leg_axis_joint" type="fixed">
+        <parent link="right_support_leg" />
+        <child link="right_support_axis" />
+        <origin xyz="0 0 ${-3/4*wheel_radius}" rpy="0 ${pi/2} 0" />
+    </joint>
+    <link name="right_support_axis">
+        <visual>
+            <origin xyz="0 0 ${wheel_thickness}" rpy="0 0 0" />
+            <geometry>
+                <cylinder length="${2*wheel_thickness}" radius="${cylindar_radius}" />
+            </geometry>
+            <material name="white" />
+        </visual>
+        <collision>
+            <origin xyz="0 0 ${wheel_thickness}" rpy="0 0 0" />
+            <geometry>
+                <cylinder length="${2*wheel_thickness}" radius="${cylindar_radius}" />
+            </geometry>
+        </collision>
+        <xacro:inertial_cylinder mass="${support_axis_mass}" length="${2*wheel_thickness}"
+            radius="${cylindar_radius}">
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
File: urdf/ros2_control.xacro (robot description, xacro)
@@ -1,58 +1,36 @@
 <?xml version="1.0"?>
 <robot name="bicycle" xmlns:xacro="http://www.ros.org/wiki/xacro">
-    <!-- TODO: teleop_twist_keyboard for bicycle (Teleoperation)? -->
-    <!-- TODO: and do a remap for topics -->
-    <!-- Hardware Interface -->
-    <!-- type="sensor" "actuator" -->
-    <!-- <ros2_control name="GazeboSimSystem" type="system"> -->
     <ros2_control name="GazeboSystem" type="system">
         <hardware>
             <plugin>gazebo_ros2_control/GazeboSystem</plugin>
-            <!-- <plugin>gz_ros2_control/GazeboSimSystem</plugin> -->
         </hardware>
-        <joint name="joint_frame_back_wheel">
+        <joint name="screw_front_wheel_joint">
+            <command_interface name="position">
+                <param name="min">-3.1415</param>
+                <param name="max">3.1415</param>
+            </command_interface>
             <command_interface name="velocity">
                 <param name="min">-10</param>
-                <param name="max">+10</param>
+                <param name="max">10</param>
             </command_interface>
+            <state_interface name="position" />
             <state_interface name="velocity" />
-            <state_interface name="position">
-                <param name="initial_value">0.0</param>
-            </state_interface>
         </joint>
-        <!-- <joint name="joint_frame_head_tube"> -->
-        <joint name="joint_fork_front_wheel">
+        <joint name="screw_back_wheel_joint">
             <command_interface name="position">
+                <param name="min">-3.1415</param>
+                <param name="max">3.1415</param>
+            </command_interface>
+            <command_interface name="velocity">
                 <param name="min">-10</param>
-                <param name="max">+10</param>
+                <param name="max">10</param>
             </command_interface>
+            <state_interface name="position" />
             <state_interface name="velocity" />
-            <state_interface name="position">
-                <param name="initial_value">0.0</param>
-            </state_interface>
         </joint>
     </ros2_control>
-    <!-- This plugins has its own controller manager. -->
-    <!-- No need to run 'ros2 run controller_manager ros2_control_node' -->
-    <!-- <gazebo>
-        <plugin name="gz_ros2_control::GazeboSimROS2ControlPlugin"
-            filename="libgz_ros2_control-system">
-            <robot_param>robot_description</robot_param>
-            <robot_param_node>robot_state_publisher</robot_param_node>
-            <parameters>
-                $(find bicycle_sim)/config/bi_controllers.yaml
-            </parameters>
-            <controller_manager_prefix_node_name>
-                controller_manager
-            </controller_manager_prefix_node_name>
-        </plugin>
-    </gazebo> -->
     <gazebo>
-        <plugin filename="libgazebo_ros2_control.so" name="gazebo_ros2_control">
-            <robot_param>robot_description</robot_param>
-            <robot_param_node>robot_state_publisher</robot_param_node>
-            <parameters>
-                $(find bicycle_sim)/config/bi_controllers.yaml
-            </parameters>
+        <plugin name="gazebo_ros2_control" filename="libgazebo_ros2_control.so">
+            <parameters>$(find bicycle_sim)/config/bicycle_controllers.yaml</parameters>
         </plugin>
     </gazebo>

Commit message: edited head tube link

File: urdf/bicycle.urdf.xacro (robot description, xacro)
@@ -47,5 +47,5 @@
     <joint name="frame_head_joint" type="revolute">
         <axis xyz="1 0 0" />
-        <limit effort="10" lower="-1.570796327" upper="+1.570796327" velocity="10" />
+        <limit effort="100" lower="-1.570796327" upper="+1.570796327" velocity="10" />
         <parent link="frame" />
         <child link="head_tube" />

Commit message: removed the colon

File: urdf/bicycle.urdf.xacro (robot description, xacro)
@@ -2,5 +2,5 @@
 <robot name="bicycle" xmlns:xacro="http://www.ros.org/wiki/xacro">
     <!-- XACRO ARG -->
-    <!-- <xacro:arg name="sim_mode" default="true" /> -->
+    <xacro:arg name="sim_mode" default="true" />
     <!-- XACRO INCLUDE -->
     <xacro:include filename="material.xacro" />

File: urdf/lidar.xacro (robot description, xacro)
@@ -48,5 +48,5 @@
                 <ros>
                     <!-- deprecated syntax -->
-                    <!-- <argument>~/out:=scan</argument> -->
+                    <!-- <argument>~/out colon=scan</argument> -->
                     <argument>--ros-args --remap ~/out:=scan</argument>
                 </ros>

File: urdf/property.xacro (robot description, xacro)
@@ -2,7 +2,7 @@
 <robot name="bicycle" xmlns:xacro="http://www.ros.org/wiki/xacro">
     <!-- XACRO PROPERTIES -->
-    <!-- TODO: thickns wheels -->
+    <!-- TODO thickns wheels -->
     <xacro:property name="wheel_radius" value="0.25" />
-    <!-- <xacro:property name="wheel_thickness" value="0.05" /> -->
+    <!-- <xacro property name="wheel_thickness" value="0.05" /> -->
     <xacro:property name="wheel_thickness" value="0.1" />
     <xacro:property name="wheel_separation" value="0.98" />

File: urdf/ros2_control.xacro (robot description, xacro)
@@ -1,5 +1,5 @@
 <?xml version="1.0"?>
 <robot name="bicycle" xmlns:xacro="http://www.ros.org/wiki/xacro">
-    <!-- TODO: Add hardware interface plugin here, and configure it -->
+    <!-- TODO Add hardware interface plugin here, and configure it -->
     <xacro:unless value="$(arg sim_mode)">
     </xacro:unless>
@@ -36,5 +36,5 @@
         <plugin name="gazebo_ros2_control" filename="libgazebo_ros2_control.so">
             <parameters>$(find bicycle_sim)/config/bicycle_controllers.yaml</parameters>
-            <!-- TODO: You may have to git clone to src -->
+            <!-- TODO  You may have to git clone to src -->
             <!-- git clone -b humble https://github.com/ros-controls/gazebo_ros2_control -->
             <!-- <parameters>$(find bicycle_sim)/config/gazebo_sim_mode.yaml</parameters> -->
